File: gpio-breakout/kicad/gpio_breakout.kicad_sch (KiCad schematic)
At the start: 12 parts, among them J1 FH41-40S-0.5SH(05), J2 Pi GPIO 2x20

Commit message: gpio-breakout A1: address design review
4-layer with solid In1 GND plane + pours (review #2), corrected FH41
land pattern 0.30x0.65 with paste margin (#4), pads 41-50 shield to
GND (#4), fused + default-bridged/cuttable 5V/3V3 links (#3), symbol
pins retyped passive (#7), fresh all-severity ERC/DRC committed (#6,
#7), J2 assembly split defined (#9), honest gate statements in README
(#2, #8). Board grown to 63.5x32 for full routing: errors-only DRC
0/0/0, zero dangling copper. Fabrication remains gated on the
interconnect contract cable identity (#1, #5).

Co-Authored-By: Claude Fable 5 <noreply@anthropic.com>
Parts:
- added F1: 0.5A polyfuse 1206, Fuse:Fuse_1206_3216Metric, symbol Device:Polyfuse
- added JP4: 5V LINK, Jumper:SolderJumper-2_P1.3mm_Bridged_RoundedPad1.0x1.5mm, symbol Jumper:SolderJumper_2_Bridged
- added JP5: 3V3 LINK, Jumper:SolderJumper-2_P1.3mm_Bridged_RoundedPad1.0x1.5mm, symbol Jumper:SolderJumper_2_Bridged
Connections:
- net +3V3: now also JP5.1 (A); no longer J1.1
- net +5V: now also JP4.1 (A); no longer J1.2, J1.4
- new net +3V3_FFC: J1.1, JP5.2 (B)
- new net +5V_FFC: F1.2, J1.2, J1.4
- new net +5V_LNK: F1.1, JP4.2 (B)
Other:
- title: koyomi gpio-breakout A0 -> koyomi gpio-breakout A1
